File: web/public/hardware/Master PCB/EEPROM.kicad_sch (KiCad schematic)
At the start: 2 parts, among them U2 M95P32-IXMNT

Commit message: Add encoder
Parts:
- added R6: 10K, symbol Device:R_Small_US
Connections:
- net +3V3: now also R6.1
- net MEM1CS: now also R6.2
Changed lines of the file:
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@@
 (kicad_sch (version 20230121) (generator eeschema)
-  (paper "A4")
-  (wire (pts (xy 121.92 97.79) (xy 132.08 97.79))
+  (paper "USLetter")
+  (junction (at 107.95 97.79) (diameter 0) (color 0 0 0 0)
+  )
+  (wire (pts (xy 107.95 97.79) (xy 132.08 97.79))
+    (stroke (width 0) (type default))
+  )
+  (wire (pts (xy 107.95 95.25) (xy 107.95 97.79))
     (stroke (width 0) (type default))
   )
@@
     (stroke (width 0) (type default))
   )
+  (wire (pts (xy 107.95 83.82) (xy 107.95 90.17))
+    (stroke (width 0) (type default))
+  )
   (wire (pts (xy 163.83 97.79) (xy 173.99 97.79))
+    (stroke (width 0) (type default))
+  )
+  (wire (pts (xy 105.41 97.79) (xy 107.95 97.79))
     (stroke (width 0) (type default))
   )
@@
     (effects (font (size 1.27 1.27)) (justify left))
   )
-  (hierarchical_label "MEM1CS" (shape input) (at 121.92 97.79 180) (fields_autoplaced)
+  (hierarchical_label "MEM1CS" (shape input) (at 105.41 97.79 180) (fields_autoplaced)
     (effects (font (size 1.27 1.27)) (justify right))
   )
@@
     )
   )
+  (symbol (lib_id "Device:R_Small_US") (at 107.95 92.71 0) (unit 1)
+    (in_bom yes) (on_board yes) (dnp no)
+    (property "Reference" "R6" (at 104.14 91.44 0)
+      (effects (font (size 1.27 1.27)) (justify left))
+    )
+    (property "Value" "10K" (at 102.87 93.98 0)
+      (effects (font (size 1.27 1.27)) (justify left))
+    )
+    (property "Footprint" "" (at 107.95 92.71 0)
+      (effects (font (size 1.27 1.27)) hide)
+    )
+    (property "Datasheet" "~" (at 107.95 92.71 0)
+      (effects (font (size 1.27 1.27)) hide)
+    )
+    (pin "1")
+    (pin "2")
+    (instances
+      (project "Master PCB"
+        (path "/61606422-4f73-4717-9ce6-6ac5e634e7ae/4dc4c3a4-08e5-49b8-a1c0-17257c3756c4"
+          (reference "R6") (unit 1)
+        )
+      )
+    )
+  )
   (symbol (lib_id "power:+3V3") (at 203.2 86.36 0) (unit 1)
     (in_bom yes) (on_board yes) (dnp no)
@@
         )
       )
+    )
+  )
+  (symbol (lib_id "power:+3V3") (at 107.95 83.82 0) (unit 1)
+    (in_bom yes) (on_board yes) (dnp no)
+    (property "Reference" "#PWR031" (at 107.95 87.63 0)
+      (effects (font (size 1.27 1.27)) hide)
+    )
+    (property "Value" "+3V3" (at 107.95 80.01 0)
+      (effects (font (size 1.27 1.27)))
+    )
+    (property "Footprint" "" (at 107.95 83.82 0)
+      (effects (font (size 1.27 1.27)) hide)
+    )
+    (property "Datasheet" "" (at 107.95 83.82 0)
+      (effects (font (size 1.27 1.27)) hide)
+    )
+    (pin "1")
+    (instances
+      (project "Master PCB"
+        (path "/61606422-4f73-4717-9ce6-6ac5e634e7ae"
+          (reference "#PWR031") (unit 1)
+        )
+        (path "/61606422-4f73-4717-9ce6-6ac5e634e7ae/4dc4c3a4-08e5-49b8-a1c0-17257c3756c4"
+          (reference "#PWR025") (unit 1)
+        )
+      )

Commit message: Finish schematic and start routing PCB
Parts:
- C16: footprint (none) -> Capacitor_SMD:C_0805_2012Metric_Pad1.18x1.45mm_HandSolder
- R6: footprint (none) -> Resistor_SMD:R_0805_2012Metric_Pad1.20x1.40mm_HandSolder
Changed lines of the file:
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@@
       (effects (font (size 1.27 1.27)) (justify left))
     )
-    (property "Footprint" "" (at 203.2 88.9 0)
+    (property "Footprint" "Capacitor_SMD:C_0805_2012Metric_Pad1.18x1.45mm_HandSolder" (at 203.2 88.9 0)
       (effects (font (size 1.27 1.27)) hide)
     )
@@
       (effects (font (size 1.27 1.27)) (justify left))
     )
-    (property "Footprint" "" (at 107.95 92.71 0)
+    (property "Footprint" "Resistor_SMD:R_0805_2012Metric_Pad1.20x1.40mm_HandSolder" (at 107.95 92.71 0)
       (effects (font (size 1.27 1.27)) hide)
     )

Commit message: More misc. cleanup and generate updated production files
Other:
- note added: "EEPROM"
Changed lines of the file:
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@@
     (stroke (width 0) (type default))
+  )
+  (rectangle (start 91.44 76.2) (end 187.96 110.49)
+    (stroke (width 0) (type default))
+    (fill (type none))
   )
   (rectangle (start 198.12 80.01) (end 214.63 96.52)
@@
     (fill (type none))
   )
+  (text "EEPROM" (at 91.44 76.2 0)
+    (effects (font (size 1.27 1.27)) (justify left bottom))
+  )
   (text "EEPROM decoupling" (at 198.12 80.01 0)
