File: web/public/hardware/Sensor PCB/Sensor PCB.kicad_pcb (KiCad board)
At the start: 2 copper layers, 65 x 60 mm, 32 parts, among them J1 Conn_01x08_Pin, J2 Conn_01x08_Pin, J3 Conn_01x02_Pin, J4 Conn_01x02_Pin, U1 DRV5033AJxDBZ, U2 DRV5033AJxDBZ, U3 DRV5033AJxDBZ, U4 DRV5033AJxDBZ, U5 74LS11, U6 74LS11

Commit message: Fixed incorrect wiring and updated PCB with new net names
Parts:
- U1, U2, U3, U4: value DRV5033AJxDBZ -> DRV5033FAQDBZR
- U5, U6: value 74LS11 -> CD74HCT11
Connections:
- net Net-(U1-OUT) renamed /HALL_OUT0
- net Net-(U2-OUT) renamed /HALL_OUT1
- net Net-(U3-OUT) renamed /HALL_OUT2
- net Net-(U4-OUT) renamed /HALL_OUT3

Commit message: Added silkscreen text to back of PCB
Other:
- board text added: "Alan Chung Ma Will Dobert Trevor Moorman Ben Owen"
- board text added: "ECE 477 Group 5 Sensor PCB Rev. A 2023-10-10"
Changed lines of the file:
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@@
   (gr_circle (center 142.5 90) (end 160 90)
     (stroke (width 0.1) (type default)) (fill none) (layer "Edge.Cuts"))
+  (gr_text "Alan Chung Ma\nWill Dobert\nTrevor Moorman\nBen Owen" (at 140.9 118.4) (layer "B.SilkS")
+    (effects (font (size 1 1) (thickness 0.2) bold) (justify left bottom mirror))
+  )
+  (gr_text "ECE 477 Group 5\nSensor PCB\nRev. A\n2023-10-10" (at 155 118.4) (layer "B.SilkS")
+    (effects (font (size 1 1) (thickness 0.2) bold) (justify left bottom mirror))
+  )
   (gr_text "GND" (at 121.9 96.3) (layer "F.SilkS")
     (effects (font (size 1 1) (thickness 0.2) bold) (justify left))

Commit message: Updated based on Ben's feedback
Removed wires between blocks, instead relying on them being connected based on net names (pained me to do this)
Fixed D3/D4 so they match the PCB layout
Renamed minor components that were previously unnamed
Parts:
- H1: value MountingHole -> Top Left Mounting Hole
- H2: value MountingHole -> Bottom Left Mounting Hole
- H3: value MountingHole -> Top Right Mounting Hole
- H4: value MountingHole -> Bottom Right Mounting Hole
- J1: value Conn_01x08_Pin -> Left Pin Header
- J2: value Conn_01x08_Pin -> Right Pin Header
- J3: value Conn_01x02_Pin -> Top Pin Header
- J4: value Conn_01x02_Pin -> Bottom Pin Header
- JP1: value SolderJumper_2_Open -> Start Row 1
- JP2: value SolderJumper_2_Open -> Start Column 1
- JP3: value SolderJumper_2_Open -> Start Column 2
- JP4: value SolderJumper_2_Open -> Start Row 2
Changed lines of the file:
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@@
         (effects (font (size 1 1) (thickness 0.15)))
     )
-    (fp_text value "MountingHole" (at 0 3.7) (layer "F.Fab")
+    (fp_text value "Top Right Mounting Hole" (at 0 3.7) (layer "F.Fab")
         (effects (font (size 1 1) (thickness 0.15)))
     )
@@
         (effects (font (size 1 1) (thickness 0.15)))
     )
-    (fp_text value "MountingHole" (at 0 3.7) (layer "F.Fab")
+    (fp_text value "Bottom Left Mounting Hole" (at 0 3.7) (layer "F.Fab")
         (effects (font (size 1 1) (thickness 0.15)))
     )
@@
         (effects (font (size 1 1) (thickness 0.15)))
     )
-    (fp_text value "SolderJumper_2_Open" (at 0 1.9 45) (layer "F.Fab")
+    (fp_text value "Start Column 1" (at 0 1.9 45) (layer "F.Fab")
         (effects (font (size 1 1) (thickness 0.15)))
     )
@@
         (effects (font (size 1 1) (thickness 0.15)))
     )
-    (fp_text value "Conn_01x08_Pin" (at 4.385 20.05) (layer "F.Fab")
+    (fp_text value "Right Pin Header" (at 4.385 20.05) (layer "F.Fab")
         (effects (font (size 1 1) (thickness 0.15)))
     )
@@
         (effects (font (size 1 1) (thickness 0.15)))
     )
-    (fp_text value "Conn_01x08_Pin" (at 4.385 20.05) (layer "F.Fab")
+    (fp_text value "Left Pin Header" (at 4.385 20.05) (layer "F.Fab")
         (effects (font (size 1 1) (thickness 0.15)))
     )
@@
         (effects (font (size 1 1) (thickness 0.15)))
     )
-    (fp_text value "Conn_01x02_Pin" (at 4.385 4.81 90) (layer "F.Fab")
+    (fp_text value "Top Pin Header" (at 4.385 4.81 90) (layer "F.Fab")
         (effects (font (size 1 1) (thickness 0.15)))
     )
@@
         (effects (font (size 1 1) (thickness 0.15)))
     )
-    (fp_text value "MountingHole" (at 0 3.7) (layer "F.Fab")
+    (fp_text value "Top Left Mounting Hole" (at 0 3.7) (layer "F.Fab")
         (effects (font (size 1 1) (thickness 0.15)))
     )
@@
         (effects (font (size 1 1) (thickness 0.15)))
     )
-    (fp_text value "SolderJumper_2_Open" (at 0 1.9 45) (layer "F.Fab")
+    (fp_text value "Start Row 2" (at 0 1.9 45) (layer "F.Fab")
         (effects (font (size 1 1) (thickness 0.15)))
     )
@@
         (effects (font (size 1 1) (thickness 0.15)))
     )
-    (fp_text value "SolderJumper_2_Open" (at 0 1.9 45) (layer "F.Fab")
+    (fp_text value "Start Row 1" (at 0 1.9 45) (layer "F.Fab")
         (effects (font (size 1 1) (thickness 0.15)))
     )
@@
         (effects (font (size 1 1) (thickness 0.15)))
     )
-    (fp_text value "Conn_01x02_Pin" (at 4.385 4.81 90) (layer "F.Fab")
+    (fp_text value "Bottom Pin Header" (at 4.385 4.81 90) (layer "F.Fab")
         (effects (font (size 1 1) (thickness 0.15)))
     )
@@
         (effects (font (size 1 1) (thickness 0.15)))
     )
-    (fp_text value "SolderJumper_2_Open" (at 0 1.9 45) (layer "F.Fab")
+    (fp_text value "Start Column 2" (at 0 1.9 45) (layer "F.Fab")
         (effects (font (size 1 1) (thickness 0.15)))
     )
@@
         (effects (font (size 1 1) (thickness 0.15)))
     )
-    (fp_text value "MountingHole" (at 0 3.7) (layer "F.Fab")
-        (effects (font (size 1 1) (thickness 0.15)))
-    )
+    (fp_text value "Bottom Right Mounting Hole" (at 0 3.7) (layer "F.Fab")
+        (effects (font (size 1 1) (thickness 0.15)))
+    )

Commit message: Change date and generate production files
Other:
- board text added: "ECE 477 Group 5 Sensor PCB Rev. A 2023-10-04"
- board text removed: "ECE 477 Group 5 Sensor PCB Rev. A 2023-10-10"
Changed lines of the file:
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@@
     (effects (font (size 1 1) (thickness 0.2) bold) (justify left bottom mirror))
   )
-  (gr_text "ECE 477 Group 5\nSensor PCB\nRev. A\n2023-10-10" (at 155 118.4) (layer "B.SilkS")
+  (gr_text "ECE 477 Group 5\nSensor PCB\nRev. A\n2023-10-04" (at 155 118.4) (layer "B.SilkS")
     (effects (font (size 1 1) (thickness 0.2) bold) (justify left bottom mirror))
   )
